File: PLL PCB - Draft.kicad_sch (KiCad schematic)
At the start: 13 parts, among them J1 Conn_01x02_Socket, J2 Conn_01x06_Socket, J4 External_VCO_RF, J5 SMA_For_External_REF

Commit message: complete pcb design
Other:
- sheet ADF4159: file ADF_OSC_LoopFilter.kicad_sch -> ADF4159.kicad_sch
Changed lines of the file:
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@@
 			)
 		)
-		(property "Sheetfile" "ADF_OSC_LoopFilter.kicad_sch"
+		(property "Sheetfile" "ADF4159.kicad_sch"
 			(at 95.25 84.4046 0)
 			(show_name no)
